File: Project/the expanse.kicad_sch (KiCad schematic)
At the start: 111 parts, among them J1 USB_C_Receptacle_USB2.0, U1 STM32F072CBT6, U2 USBLC6-2SC6

Commit message: Added ISO, stitched GND plane, cleaned up repo files
Parts:
- added MX46: MX_SW_solder, PCM_marbastlib-mx:SW_MX_1.25u, symbol PCM_marbastlib-mx:MX_SW_solder
- added S5: ISO, PCM_marbastlib-mx:STAB_MX_P_ISO-ROT, symbol PCM_marbastlib-mx:MX_stab
Connections:
- net COL11: now also MX46.2
- net at D24.2 (A), MX24.1: now also MX46.1
